File: electronics/view_screen/view_screen.kicad_sch (KiCad schematic)
At the start: 12 parts, among them J1 Conn_01x04, J2 GC9A01, J3 Conn_01x04, J4 Conn_01x04, J5 Conn_01x04, Q1 2N7002

Commit message: Initial start
Parts:
- C1: footprint Capacitor_SMD:C_0805_2012Metric -> Capacitor_SMD:C_0603_1608Metric
- C2: footprint Capacitor_SMD:C_0603_1608Metric -> Capacitor_SMD:C_0402_1005Metric
- R1, R2, R3: footprint Resistor_SMD:R_0603_1608Metric -> Resistor_SMD:R_0402_1005Metric
